File: OOS - optyczny odbiornik sygnalow/Sekcja_USB.kicad_sch (KiCad schematic)
At the start: 12 parts, among them J6 USB_C_Receptacle

Commit message: Adding max board dimentions possible to get 2$ PCBs from JLCPCB. Dimentions will be shrunk as the components are being placed
Parts:
- C24: value 1u -> 100n; MPN CC0603KRX7R7BB105 -> CL10B104KO8WPNC; Supplier Link https://www.tme.eu/pl/details/cc0603krx7r7bb105/kondensator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 -> https://www.tme.eu/pl/details/cl10b104ko8wpnc/kondensatory-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
Connections:
- net +5V: now also C24.1; no longer C23.1
- net C24_net: now also C23.1; no longer C24.1
Other:
- moved on the sheet: C23
Changed lines of the file:
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@@
 			"AEpKIJE0RojVajBMY4qhOQ4cR0rpCAQQISYQCIQWh4QmCAQCoYUhQkwgEAgtDBFiAoFAaGGIEBMI"
 			"BEILQ4SYQCAQWhgixAQCgdDCECEmEAiEFoYIMYFAILQwRIgJBAKhhSFCTCAQCC3M/wEWgIiQzR52"
-			"UwAAAABJRU5ErkJggg=="
+			"UwAAAABJRU5ErkJgggAAAAAAAAAAAAAAAAAAAAAAAAAAAOsti6kAHgiAAAAAAAAAAAAAAAAAAAAA"
+			"AAAAAAAAAAAA6S2JqQAfCIAAAAAAAAAAAAAAAAAAAAAAAAAAAAAAAADnLY+pACAIgAAAAAAAAAAA"
+			"AAAAAAAAAAAAAAAAAAAAAOUtjakAIQiAAAAAAAAAAAAAAAAAAAAAAAAAAAAAAAAA4y2DqQAiCIAA"
+			"AAAAAAAAAAAAAAAAAAAAAAAAAAAAAADhLYGpACMIgAAAAAAAAAAAAAAAAAAAAAAAAAAAAAAAAN8t"
+			"h6kAJAiAAAAAAAAAAAAAAAAAAAAAAAAAAAAAAAAA3S2FqQAlCIAAAAAAAAAAAAAAAAAAAAAAAAAA"
+			"AAAAAADbLbupACYIgAAAAAAAAAAAAAAAAAAAAAAAAAAAAAAAANktuakAJwiAAAAAAAAAAAAAAAAA"
+			"AAAAAAAAAAAAAAAA1y2/qQAoCIAAAAAAAAAAAAAAAAAAAAAAAAAAAAAAAADVLb2pACkIgAAAAAAA"
+			"AAAAAAAAAAAAAAAAAAAAAAAAANMts6kAKgiAAAAAAAAAAAAAAAAAAAAAAAAAAAAAAAAA0S2xqQAr"
+			"CIAAAAAAAAAAAAAAAAAAAAAAAAAAAAAAAADPLbepACwIgAAAAAAAAAAAAAAAAAAAAAAAAAAAAAAA"
+			"AM0ttakALQiAAAAAAAAAAAAAAAAAAAAAAAAAAAAAAAAAyy2rqQAuCIAAAAAAAAAAAAAAAAAAAAAA"
+			"AAAAAAAAAADJLampAC8IgAAAAAAAAAAAAAAAAAAAAAAAAAAAAAAAAMctr6kAMAiAAAAAAAAAAAAA"
+			"AAAAAAAAAAAAAAAAAAAAxS2tqQAxCIAAAAAAAAAAAAAAAAAAAAAAAAAAAAAAAADDLaOpADIIgAAA"
+			"AAAAAAAAAAAAAAAAAAAAAAAAAAAAAMEtoakAMwiAAAAAAAAAAAAAAAAAAAAAAAAAAAAAAAAAPy2n"
+			"qQA0CIAAAAAAAAAAAAAAAAAAAAAAAAAAAAAAAAA9LaWpADUIgAAAAAAAAAAAAAAAAAAAAAAAAAAA"
+			"AAAAADstW6kANgiAAAAAAAAAAAAAAAAAAAAAAAAAAAAAAAAAOS1ZqQA3CIAAAAAAAAAAAAAAAAAA"
+			"AAAAAAAAAAAAAAA3LV+pADgIgAAAAAAAAAAAAAAAAAAAAAAAAAAAAAAAADUtXakAOQiAAAAAAAAA"
+			"AAAAAAAAAAAAAAAAAAAAAAAAMy1TqQA6CIAAAAAAAAAAAAAAAAAAAAAAAAAAAAAAAAAxLVGpADsI"
+			"gAAAAAAAAAAAAAAAAAAAAAAAAAAAAAAAAC8tV6kAPAiAAAAAAAAAAAAAAAAAAAAAAAAAAAAAAAAA"
+			"LS1VqQA9CIAAAAAAAA=="
 		)
 	)
@@
 	(symbol
 		(lib_id "Device:C")
-		(at 228.6 66.04 0)
+		(at 204.47 66.04 0)
 		(unit 1)
 		(exclude_from_sim no)
@@
 		(dnp no)
 		(property "Reference" "C23"
-			(at 231.14 63.5 0)
+			(at 207.01 63.5 0)
 			(effects
 				(font
@@
 		)
 		(property "Value" "10u"
-			(at 231.14 64.77 0)
+			(at 207.01 64.77 0)
 			(effects
 				(font
@@
 		)
 		(property "Footprint" "Capacitor_SMD:C_1210_3225Metric_Pad1.33x2.70mm_HandSolder"
-			(at 229.5652 69.85 0)
+			(at 205.4352 69.85 0)
 			(effects
 				(font
@@
 		)
 		(property "Datasheet" "https://www.tme.eu/Document/6e14d5d12404104c8b499de9805d45d5/CGA-series.pdf"
-			(at 228.6 66.04 0)
+			(at 204.47 66.04 0)
 			(effects
 				(font
@@
 		)
 		(property "Description" "Unpolarized ceramic capacitor"
-			(at 228.6 66.04 0)
+			(at 204.47 66.04 0)
 			(effects
 				(font
@@
 		)
 		(property "Voltage Rating" "75V"
-			(at 231.14 66.04 0)
+			(at 207.01 66.04 0)
 			(effects
 				(font
@@
 		)
 		(property "Dielectric" "X7R"
-			(at 231.14 67.31 0)
+			(at 207.01 67.31 0)
 			(effects
 				(font
@@
 		)
 		(property "Package" "1210"
-			(at 228.6 66.04 0)
+			(at 204.47 66.04 0)
 			(effects
 				(font
@@
 		)
 		(property "Tolerance" "±10%"
-			(at 231.14 68.58 0)
+			(at 207.01 68.58 0)
 			(effects
 				(font
@@
 		)
 		(property "Supplier" "TME"
-			(at 228.6 66.04 0)
+			(at 204.47 66.04 0)
 			(effects
 				(font
@@
 		)
 		(property "Supplier Link" "https://www.tme.eu/pl/en/details/cga6p1x7r1n106kac/mlcc-smd-capacitors/tdk/cga6p1x7r1n106k250ac/"
-			(at 228.6 66.04 0)
+			(at 204.47 66.04 0)
 			(effects
 				(font
@@
 	(symbol
 		(lib_id "Device:C")
-		(at 204.47 66.04 0)
+		(at 228.6 66.04 0)
 		(unit 1)
 		(exclude_from_sim no)
@@
 		(dnp no)
 		(property "Reference" "C24"
-			(at 207.01 63.5 0)
-			(effects
-				(font
-					(size 0.762 0.762)
-				)
-				(justify left)
-			)
-		)
-		(property "Value" "1u"
-			(at 207.01 64.77 0)
+			(at 231.14 63.5 0)
+			(effects
+				(font
+					(size 0.762 0.762)
+				)
+				(justify left)
+			)
+		)
+		(property "Value" "100n"
+			(at 231.14 64.77 0)
 			(effects
 				(font
@@
 		)
 		(property "Footprint" "Capacitor_SMD:C_0603_1608Metric_Pad1.08x0.95mm_HandSolder"
-			(at 205.4352 69.85 0)
-			(effects
-				(font
-					(size 0.762 0.762)
-				)
-				(justify left)
-				(hide yes)
-			)
-		)
-		(property "Datasheet" "https://www.yageo.com/upload/media/product/productsearch/datasheet/mlcc/UPY-GPHC_X7R_6.3V-to-250V_26.pdf"
-			(at 204.47 66.04 0)
+			(at 229.5652 69.85 0)
+			(effects
+				(font
+					(size 0.762 0.762)
+				)
+				(justify left)
+				(hide yes)
+			)
+		)
+		(property "Datasheet" "https://www.tme.eu/Document/7da762c1dbaf553c64ad9c40d3603826/mlcc_samsung.pdf"
+			(at 228.6 66.04 0)
 			(effects
 				(font
@@
 		)
 		(property "Description" "Unpolarized capacitor"
-			(at 204.47 66.04 0)
+			(at 228.6 66.04 0)
 			(effects
 				(font
@@
 		)
 		(property "Voltage Rating" "16V"
-			(at 207.01 66.04 0)
+			(at 231.14 66.04 0)
 			(effects
 				(font
@@
 		)
 		(property "Dielectric" "X7R"
-			(at 207.01 67.31 0)
+			(at 231.14 67.31 0)
 			(effects
 				(font
@@
 		)
 		(property "Package" "0603"
-			(at 204.47 66.04 0)
-			(effects
-				(font
-					(size 0.762 0.762)
-				)
+			(at 228.6 66.04 0)
+			(effects
+				(font
+					(size 0.762 0.762)
+				)
+			)
+		)
+		(property "Tolerance" "±10%"
+			(at 231.14 68.58 0)
+			(effects
+				(font
+					(size 0.762 0.762)
+				)
+				(justify left)
 			)
 		)
 		(property "Supplier" "TME"
-			(at 204.47 66.04 0)
-			(effects
-				(font
-					(size 0.762 0.762)
-				)
-				(hide yes)
-			)
-		)
-		(property "Tolerance" "±10%"
-			(at 207.01 68.58 0)
-			(effects
-				(font
-					(size 0.762 0.762)
-				)
-				(justify left)
-			)
-		)
-		(property "MPN" "CC0603KRX7R7BB105"
-			(at 204.47 66.04 0)
-			(effects
-				(font
-					(size 0.762 0.762)
-				)
-				(hide yes)
-			)
-		)
-		(property "Supplier Link" "https://www.tme.eu/pl/details/cc0603krx7r7bb105/kondensatory-mlcc-smd/yageo/"
-			(at 204.47 66.04 0)
-			(effects
-				(font
+			(at 228.6 66.04 0)
+			(effects
+				(font
+					(size 0.762 0.762)
+				)
+				(hide yes)
+			)
+		)
+		(property "MPN" "CL10B104KO8WPNC"
+			(at 228.6 66.04 0)
+			(effects
+				(font
+					(size 0.762 0.762)
+				)
+				(hide yes)
+			)
+		)
+		(property "Supplier Link" "https://www.tme.eu/pl/details/cl10b104ko8wpnc/kondensatory-mlcc-smd/samsung/"
+			(at 228.6 66.04 0)
+			(effects
+				(font

Commit message: Added polygon for USB3.2, move TP37 on a schematic
Connections:
- net C24_net: no longer TP37.1
- net J6_Vbus: now also TP37.1
Other:
- moved on the sheet: TP37
Changed lines of the file:
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@@
+	)
+	(junction
+		(at 176.53 60.96)
+		(diameter 0)
+		(color 0 0 0 0)
 	)
 	(junction
@@
 	)
 	(junction
-		(at 190.5 60.96)
-		(diameter 0)
-		(color 0 0 0 0)
-	)
-	(junction
 		(at 171.45 58.42)
 		(diameter 0)
@@
 	)
 	(junction
+		(at 190.5 60.96)
+		(diameter 0)
+		(color 0 0 0 0)
+	)
+	(junction
 		(at 151.13 128.27)
 		(diameter 0)
@@
 	(wire
 		(pts
+			(xy 176.53 60.96) (xy 180.34 60.96)
+		)
+		(stroke
+			(width 0)
+			(type default)
+		)
+	)
+	(wire
+		(pts
 			(xy 204.47 60.96) (xy 204.47 62.23)
 		)
@@
 	(wire
 		(pts
-			(xy 171.45 60.96) (xy 180.34 60.96)
+			(xy 171.45 60.96) (xy 176.53 60.96)
 		)
 		(stroke
@@
 	)
 	(label "J6_Vbus"
-		(at 173.99 60.96 0)
+		(at 172.085 60.96 0)
 		(effects
 			(font
@@
 	(symbol
 		(lib_id "Connector:TestPoint_Small")
-		(at 190.5 60.96 0)
+		(at 176.53 60.96 0)
 		(unit 1)
 		(exclude_from_sim no)
@@
 		(dnp no)
 		(property "Reference" "TP37"
-			(at 190.5 59.69 0)
+			(at 176.53 59.69 0)
 			(effects
 				(font
@@
 		)
 		(property "Value" "TestPoint_Small"
-			(at 191.77 62.2299 0)
+			(at 177.8 62.2299 0)
 			(effects
 				(font
@@
 		)
 		(property "Footprint" "TestPoint:TestPoint_Pad_D1.0mm"
-			(at 195.58 60.96 0)
+			(at 181.61 60.96 0)
 			(effects
 				(font
@@
 		)
 		(property "Datasheet" "~"
-			(at 195.58 60.96 0)
+			(at 181.61 60.96 0)
 			(effects
 				(font
@@
 		)
 		(property "Description" "test point"
-			(at 190.5 60.96 0)
-			(effects
-				(font
+			(at 176.53 60.96 0)
+			(effects
+				(font

Commit message: Moved TP37 on schematic, Added LED diode with resistor for +5V indication, improved component placement for USB3.2
Parts:
- added D8: LED, Diode_SMD:D_0603_1608Metric_Pad1.05x0.95mm_HandSolder, symbol Device:LED
- added R27: 2k2, Resistor_SMD:R_0603_1608Metric_Pad0.98x0.95mm_HandSolder, symbol Device:R
- added TP39: TestPoint_Small, TestPoint:TestPoint_Pad_D1.0mm, symbol Connector:TestPoint_Small
Connections:
- net +5V: now also C23.1, R27.1; no longer C24.1
- net 0V: now also D8.1 (K)
- net C24_net: now also C24.1; no longer C23.1
- new net: D8.2 (A), R27.2, TP39.1
Other:
- moved on the sheet: C23, C24
