File: OOS - optyczny odbiornik sygnalow/Sekcja_USB.kicad_sch (KiCad schematic)
At the start: 15 parts, among them J6 USB_C_Receptacle

Commit message: Dodane napisy na jumperach
Parts:
- J6: footprint Connector_USB:USB_C_Receptacle_Amphenol_12401548E4-2A -> USB_connectors:USB_C_Receptacle_Amphenol_12401548E4-2A
Changed lines of the file:
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@@
 			)
 		)
-		(property "Footprint" "Connector_USB:USB_C_Receptacle_Amphenol_12401548E4-2A"
+		(property "Footprint" "USB_connectors:USB_C_Receptacle_Amphenol_12401548E4-2A"
 			(at 157.48 86.36 0)
 			(effects
